File: pcb/rev1/rfamp.brd (EAGLE design)
At the start: 40 x 20 mm, 17 parts, among them IC1 TS520530, IC2 ADL5523, X1 SAW-B3721

Commit message: Minor changes.
Parts:
- MOV1: value MOV -> (none)
- renumbered R1 to MOV1
Changed lines of the file:
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@@
 <grid distance="0.2" unitdist="mm" unit="mm" style="lines" multiple="1" display="no" altdistance="0.2" altunitdist="mm" altunit="mm"/>
 <layers>
-<layer number="1" name="Top" color="4" fill="1" visible="no" active="yes"/>
-<layer number="16" name="Bottom" color="1" fill="1" visible="no" active="yes"/>
+<layer number="1" name="Top" color="4" fill="1" visible="yes" active="yes"/>
+<layer number="16" name="Bottom" color="1" fill="1" visible="yes" active="yes"/>
 <layer number="17" name="Pads" color="2" fill="1" visible="yes" active="yes"/>
 <layer number="18" name="Vias" color="2" fill="1" visible="yes" active="yes"/>
@@
 <layer number="20" name="Dimension" color="15" fill="1" visible="yes" active="yes"/>
 <layer number="21" name="tPlace" color="7" fill="1" visible="no" active="yes"/>
-<layer number="22" name="bPlace" color="7" fill="1" visible="yes" active="yes"/>
+<layer number="22" name="bPlace" color="7" fill="1" visible="no" active="yes"/>
 <layer number="23" name="tOrigins" color="15" fill="1" visible="no" active="yes"/>
-<layer number="24" name="bOrigins" color="15" fill="1" visible="yes" active="yes"/>
+<layer number="24" name="bOrigins" color="15" fill="1" visible="no" active="yes"/>
 <layer number="25" name="tNames" color="7" fill="1" visible="no" active="yes"/>
-<layer number="26" name="bNames" color="7" fill="1" visible="yes" active="yes"/>
+<layer number="26" name="bNames" color="7" fill="1" visible="no" active="yes"/>
 <layer number="27" name="tValues" color="7" fill="1" visible="no" active="yes"/>
 <layer number="28" name="bValues" color="7" fill="1" visible="no" active="yes"/>
 <layer number="29" name="tStop" color="7" fill="3" visible="no" active="yes"/>
-<layer number="30" name="bStop" color="7" fill="6" visible="yes" active="yes"/>
+<layer number="30" name="bStop" color="7" fill="6" visible="no" active="yes"/>
 <layer number="31" name="tCream" color="7" fill="4" visible="no" active="yes"/>
 <layer number="32" name="bCream" color="7" fill="5" visible="no" active="yes"/>
@@
 <layer number="46" name="Milling" color="3" fill="1" visible="no" active="yes"/>
 <layer number="47" name="Measures" color="7" fill="1" visible="no" active="yes"/>
-<layer number="48" name="Document" color="7" fill="1" visible="yes" active="yes"/>
+<layer number="48" name="Document" color="7" fill="1" visible="no" active="yes"/>
 <layer number="49" name="Reference" color="7" fill="1" visible="no" active="yes"/>
 <layer number="50" name="dxf" color="7" fill="1" visible="no" active="yes"/>
 <layer number="51" name="tDocu" color="7" fill="1" visible="no" active="yes"/>
-<layer number="52" name="bDocu" color="7" fill="1" visible="yes" active="yes"/>
+<layer number="52" name="bDocu" color="7" fill="1" visible="no" active="yes"/>
 <layer number="53" name="tGND_GNDA" color="7" fill="9" visible="no" active="no"/>
 <layer number="54" name="bGND_GNDA" color="1" fill="9" visible="no" active="no"/>
@@
 <attribute name="VALUE" x="13.2" y="10" size="1.016" layer="27" font="vector" ratio="15" rot="R90"/>
 </element>
-<element name="R1" library="rcl" package="R0603" value="MOV" x="6" y="5.6" smashed="yes" rot="R90">
-<attribute name="NAME" x="7.2" y="4" size="1.016" layer="25" font="vector" ratio="15" rot="R180"/>
+<element name="MOV1" library="rcl" package="R0603" value="" x="6" y="5.6" smashed="yes" rot="R90">
+<attribute name="NAME" x="8.6" y="4" size="1.016" layer="25" font="vector" ratio="15" rot="R180"/>
 <attribute name="VALUE" x="7.905" y="4.965" size="1.27" layer="27" rot="R90"/>
 </element>
@@
 <contactref element="X1" pad="1"/>
 <contactref element="X1" pad="4"/>
-<contactref element="R1" pad="1"/>
+<contactref element="MOV1" pad="1"/>
 <via x="5.2" y="4.6" extent="1-16" drill="0.3"/>
 <via x="6.6" y="4.6" extent="1-16" drill="0.3"/>
@@
 <signal name="N$1" class="1">
 <contactref element="RFIN" pad="1"/>
-<contactref element="R1" pad="2"/>
+<contactref element="MOV1" pad="2"/>
 <contactref element="X1" pad="2"/>
 <wire x1="2.3154" y1="7" x2="6" y2="7" width="2.4" layer="1"/>

Commit message: Fix board outline (move SMA conenctors to board edges).
Parts:
- moved RFOUT 0.20 mm to (40.0, 7.00)
- moved RFIN 0.20 mm to (0.00, 7.00)
Routing:
- net GND: track 6.00 -> 14.0 mm
Changed lines of the file:
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@@
 <layer number="19" name="Unrouted" color="6" fill="1" visible="yes" active="yes"/>
 <layer number="20" name="Dimension" color="15" fill="1" visible="yes" active="yes"/>
-<layer number="21" name="tPlace" color="7" fill="1" visible="no" active="yes"/>
+<layer number="21" name="tPlace" color="7" fill="1" visible="yes" active="yes"/>
 <layer number="22" name="bPlace" color="7" fill="1" visible="no" active="yes"/>
-<layer number="23" name="tOrigins" color="15" fill="1" visible="no" active="yes"/>
+<layer number="23" name="tOrigins" color="15" fill="1" visible="yes" active="yes"/>
 <layer number="24" name="bOrigins" color="15" fill="1" visible="no" active="yes"/>
-<layer number="25" name="tNames" color="7" fill="1" visible="no" active="yes"/>
+<layer number="25" name="tNames" color="7" fill="1" visible="yes" active="yes"/>
 <layer number="26" name="bNames" color="7" fill="1" visible="no" active="yes"/>
 <layer number="27" name="tValues" color="7" fill="1" visible="no" active="yes"/>
@@
 </autorouter>
 <elements>
-<element name="RFIN" library="con-coax" package="J502-ND-142-0711-821/826" value="" x="0.2" y="7" smashed="yes">
-<attribute name="OC_NEWARK" value="16F3627" x="0.2" y="7" size="1.778" layer="27" display="off"/>
-<attribute name="MPN" value="142-0711-821" x="0.2" y="7" size="1.778" layer="27" display="off"/>
-<attribute name="MF" value="JOHNSON COMPONENTS" x="0.2" y="7" size="1.778" layer="27" display="off"/>
-<attribute name="OC_FARNELL" value="1019328" x="0.2" y="7" size="1.778" layer="27" display="off"/>
-<attribute name="NAME" x="5" y="10.4" size="1.016" layer="25" font="vector" ratio="15"/>
-<attribute name="VALUE" x="1.47" y="-1.89" size="1.778" layer="27"/>
-</element>
-<element name="RFOUT" library="con-coax" package="J502-ND-142-0711-821/826" value="" x="39.8" y="7" smashed="yes" rot="R180">
-<attribute name="OC_NEWARK" value="16F3627" x="39.8" y="7" size="1.778" layer="27" rot="R180" display="off"/>
-<attribute name="MPN" value="142-0711-821" x="39.8" y="7" size="1.778" layer="27" rot="R180" display="off"/>
-<attribute name="MF" value="JOHNSON COMPONENTS" x="39.8" y="7" size="1.778" layer="27" rot="R180" display="off"/>
-<attribute name="OC_FARNELL" value="1019328" x="39.8" y="7" size="1.778" layer="27" rot="R180" display="off"/>
-<attribute name="NAME" x="35.2" y="4" size="1.016" layer="25" font="vector" ratio="15" rot="R180"/>
-<attribute name="VALUE" x="38.53" y="15.89" size="1.778" layer="27" rot="R180"/>
+<element name="RFIN" library="con-coax" package="J502-ND-142-0711-821/826" value="" x="0" y="7" smashed="yes">
+<attribute name="OC_NEWARK" value="16F3627" x="0" y="7" size="1.778" layer="27" display="off"/>
+<attribute name="MPN" value="142-0711-821" x="0" y="7" size="1.778" layer="27" display="off"/>
+<attribute name="MF" value="JOHNSON COMPONENTS" x="0" y="7" size="1.778" layer="27" display="off"/>
+<attribute name="OC_FARNELL" value="1019328" x="0" y="7" size="1.778" layer="27" display="off"/>
+<attribute name="NAME" x="4.8" y="10.4" size="1.016" layer="25" font="vector" ratio="15"/>
+<attribute name="VALUE" x="1.27" y="-1.89" size="1.778" layer="27"/>
+</element>
+<element name="RFOUT" library="con-coax" package="J502-ND-142-0711-821/826" value="" x="40" y="7" smashed="yes" rot="R180">
+<attribute name="OC_NEWARK" value="16F3627" x="40" y="7" size="1.778" layer="27" rot="R180" display="off"/>
+<attribute name="MPN" value="142-0711-821" x="40" y="7" size="1.778" layer="27" rot="R180" display="off"/>
+<attribute name="MF" value="JOHNSON COMPONENTS" x="40" y="7" size="1.778" layer="27" rot="R180" display="off"/>
+<attribute name="OC_FARNELL" value="1019328" x="40" y="7" size="1.778" layer="27" rot="R180" display="off"/>
+<attribute name="NAME" x="35.4" y="4" size="1.016" layer="25" font="vector" ratio="15" rot="R180"/>
+<attribute name="VALUE" x="38.73" y="15.89" size="1.778" layer="27" rot="R180"/>
 </element>
 <element name="X1" library="qyx-misc" package="B3721" value="SAW-B3721" x="12.2" y="7" smashed="yes" rot="R90">
@@
 <contactref element="POWER" pad="C"/>
 <via x="15.8" y="16.4" extent="1-16" drill="0.3"/>
-<wire x1="38" y1="9.4" x2="39.4" y2="9.4" width="0" layer="19" extent="1-1"/>
-<wire x1="36.6" y1="9.4" x2="35.2" y2="9.4" width="0" layer="19" extent="1-1"/>
-<wire x1="39.4" y1="4.6" x2="38" y2="4.6" width="0" layer="19" extent="1-1"/>
-<wire x1="36.6" y1="4.6" x2="35.2" y2="4.6" width="0" layer="19" extent="1-1"/>
+<wire x1="36.6" y1="9.4" x2="38" y2="9.4" width="0.2" layer="1"/>
+<wire x1="38" y1="9.4" x2="39.4" y2="9.4" width="0.2" layer="1"/>
+<wire x1="37.8846" y1="10.4946" x2="38" y2="10.4946" width="0.2" layer="1"/>
+<wire x1="38" y1="10.4946" x2="38" y2="9.4" width="0.2" layer="1"/>
+<wire x1="36.6" y1="4.6" x2="38" y2="4.6" width="0.2" layer="1"/>
+<wire x1="38" y1="4.6" x2="37.8846" y2="4.6" width="0.2" layer="1"/>
+<wire x1="37.8846" y1="4.6" x2="37.8846" y2="3.5054" width="0.2" layer="1"/>
+<wire x1="38" y1="4.6" x2="39.4" y2="4.6" width="0.2" layer="1"/>
 </signal>
 <signal name="N$1" class="1">
@@
 <contactref element="MOV1" pad="2"/>
 <contactref element="X1" pad="2"/>
-<wire x1="2.3154" y1="7" x2="6" y2="7" width="2.4" layer="1"/>
+<wire x1="2.1154" y1="7" x2="6" y2="7" width="2.4" layer="1"/>
 <wire x1="6" y1="7" x2="8.8" y2="7" width="2.4" layer="1"/>
 <wire x1="8.8" y1="7" x2="10.9" y2="7" width="0.6096" layer="1"/>
@@
 <wire x1="28.9" y1="7.05" x2="30.95" y2="7.05" width="0.3" layer="1"/>
 <wire x1="30.95" y1="7.05" x2="31" y2="7" width="0.3" layer="1"/>
-<wire x1="31" y1="7" x2="37.6846" y2="7" width="2.4" layer="1"/>
+<wire x1="31" y1="7" x2="37.8846" y2="7" width="2.4" layer="1"/>
 </signal>
 <signal name="+5V">

Commit message: Replace SMA edge connectors.
Parts:
- removed RFIN, RFOUT: (no value), con-coax:J502-ND-142-0711-821/826
- added J$1, J$2: SMA_EDGE, SparkFun:SMA-EDGE
Connections:
- net GND: now also J$1.GND@0, J$1.GND@1, J$1.GND@2, J$1.GND@3, J$2.GND@0, J$2.GND@1, J$2.GND@2, J$2.GND@3; no longer RFIN.G@1, RFIN.G@2, RFIN.G@3, RFIN.G@4, RFOUT.G@1, RFOUT.G@2, RFOUT.G@3, RFOUT.G@4
- net N$1: now also J$1.SIG; no longer RFIN.1
- net N$6: now also J$2.SIG; no longer RFOUT.1
Routing:
- net GND: track 14.0 -> 6.00 mm, vias 95 -> 93
Changed lines of the file:
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@@
 </autorouter>
 <elements>
-<element name="RFIN" library="con-coax" package="J502-ND-142-0711-821/826" value="" x="0" y="7" smashed="yes">
-<attribute name="OC_NEWARK" value="16F3627" x="0" y="7" size="1.778" layer="27" display="off"/>
-<attribute name="MPN" value="142-0711-821" x="0" y="7" size="1.778" layer="27" display="off"/>
-<attribute name="MF" value="JOHNSON COMPONENTS" x="0" y="7" size="1.778" layer="27" display="off"/>
-<attribute name="OC_FARNELL" value="1019328" x="0" y="7" size="1.778" layer="27" display="off"/>
-<attribute name="NAME" x="4.8" y="10.4" size="1.016" layer="25" font="vector" ratio="15"/>
-<attribute name="VALUE" x="1.27" y="-1.89" size="1.778" layer="27"/>
-</element>
-<element name="RFOUT" library="con-coax" package="J502-ND-142-0711-821/826" value="" x="40" y="7" smashed="yes" rot="R180">
-<attribute name="OC_NEWARK" value="16F3627" x="40" y="7" size="1.778" layer="27" rot="R180" display="off"/>
-<attribute name="MPN" value="142-0711-821" x="40" y="7" size="1.778" layer="27" rot="R180" display="off"/>
-<attribute name="MF" value="JOHNSON COMPONENTS" x="40" y="7" size="1.778" layer="27" rot="R180" display="off"/>
-<attribute name="OC_FARNELL" value="1019328" x="40" y="7" size="1.778" layer="27" rot="R180" display="off"/>
-<attribute name="NAME" x="35.4" y="4" size="1.016" layer="25" font="vector" ratio="15" rot="R180"/>
-<attribute name="VALUE" x="38.73" y="15.89" size="1.778" layer="27" rot="R180"/>
-</element>
 <element name="X1" library="qyx-misc" package="B3721" value="SAW-B3721" x="12.2" y="7" smashed="yes" rot="R90">
 <attribute name="NAME" x="13.2" y="4" size="1.016" layer="25" font="vector" ratio="15" rot="R180"/>
@@
 <attribute name="VALUE" x="15.095" y="17.67" size="1.27" layer="27" rot="R270"/>
 </element>
+<element name="J$1" library="SparkFun" package="SMA-EDGE" value="SMA_EDGE" x="2.4" y="4.45" rot="R90"/>
+<element name="J$2" library="SparkFun" package="SMA-EDGE" value="SMA_EDGE" x="37.6" y="4.45" rot="R90"/>
 </elements>
 <signals>
@@
 </polygon>
 <via x="0.8" y="1.2" extent="1-16" drill="0.3"/>
-<contactref element="RFIN" pad="G@4"/>
-<contactref element="RFIN" pad="G@3"/>
-<contactref element="RFIN" pad="G@1"/>
-<contactref element="RFIN" pad="G@2"/>
-<contactref element="RFOUT" pad="G@4"/>
-<contactref element="RFOUT" pad="G@3"/>
-<contactref element="RFOUT" pad="G@1"/>
-<contactref element="RFOUT" pad="G@2"/>
 <contactref element="X1" pad="3"/>
 <contactref element="X1" pad="6"/>
@@
 <via x="27.4" y="7.4" extent="1-16" drill="0.3"/>
 <via x="27.4" y="6.2" extent="1-16" drill="0.3"/>
-<via x="31" y="9.4" extent="1-16" drill="0.3"/>
-<via x="32.4" y="9.4" extent="1-16" drill="0.3"/>
-<via x="33.8" y="9.4" extent="1-16" drill="0.3"/>
-<via x="31" y="4.6" extent="1-16" drill="0.3"/>
-<via x="32.4" y="4.6" extent="1-16" drill="0.3"/>
-<via x="33.8" y="4.6" extent="1-16" drill="0.3"/>
-<via x="35.2" y="4.6" extent="1-16" drill="0.3"/>
-<via x="35.2" y="9.4" extent="1-16" drill="0.3"/>
-<via x="36.6" y="9.4" extent="1-16" drill="0.3"/>
-<via x="38" y="9.4" extent="1-16" drill="0.3"/>
-<via x="39.4" y="9.4" extent="1-16" drill="0.3"/>
-<via x="36.6" y="4.6" extent="1-16" drill="0.3"/>
-<via x="38" y="4.6" extent="1-16" drill="0.3"/>
-<via x="39.4" y="4.6" extent="1-16" drill="0.3"/>
+<via x="31.2" y="9.4" extent="1-16" drill="0.3"/>
+<via x="32.8" y="9.4" extent="1-16" drill="0.3"/>
+<via x="34.4" y="9.4" extent="1-16" drill="0.3"/>
+<via x="31.2" y="4.6" extent="1-16" drill="0.3"/>
+<via x="32.8" y="4.6" extent="1-16" drill="0.3"/>
+<via x="34.4" y="4.6" extent="1-16" drill="0.3"/>
+<via x="36" y="4.6" extent="1-16" drill="0.3"/>
+<via x="36" y="9.4" extent="1-16" drill="0.3"/>
 <via x="3.8" y="9.4" extent="1-16" drill="0.3"/>
 <via x="2.4" y="9.4" extent="1-16" drill="0.3"/>
@@
 <contactref element="POWER" pad="C"/>
 <via x="15.8" y="16.4" extent="1-16" drill="0.3"/>
-<wire x1="36.6" y1="9.4" x2="38" y2="9.4" width="0.2" layer="1"/>
-<wire x1="38" y1="9.4" x2="39.4" y2="9.4" width="0.2" layer="1"/>
-<wire x1="37.8846" y1="10.4946" x2="38" y2="10.4946" width="0.2" layer="1"/>
-<wire x1="38" y1="10.4946" x2="38" y2="9.4" width="0.2" layer="1"/>
-<wire x1="36.6" y1="4.6" x2="38" y2="4.6" width="0.2" layer="1"/>
-<wire x1="38" y1="4.6" x2="37.8846" y2="4.6" width="0.2" layer="1"/>
-<wire x1="37.8846" y1="4.6" x2="37.8846" y2="3.5054" width="0.2" layer="1"/>
-<wire x1="38" y1="4.6" x2="39.4" y2="4.6" width="0.2" layer="1"/>
+<contactref element="J$1" pad="GND@3"/>
+<contactref element="J$1" pad="GND@2"/>
+<contactref element="J$1" pad="GND@1"/>
+<contactref element="J$1" pad="GND@0"/>
+<contactref element="J$2" pad="GND@3"/>
+<contactref element="J$2" pad="GND@2"/>
+<contactref element="J$2" pad="GND@1"/>
+<contactref element="J$2" pad="GND@0"/>
+<via x="37.6" y="9.4" extent="1-16" drill="0.3"/>
+<via x="39" y="9.4" extent="1-16" drill="0.3"/>
+<via x="37.6" y="4.6" extent="1-16" drill="0.3"/>
+<via x="39" y="4.6" extent="1-16" drill="0.3"/>
 </signal>
 <signal name="N$1" class="1">
-<contactref element="RFIN" pad="1"/>
 <contactref element="MOV1" pad="2"/>
 <contactref element="X1" pad="2"/>
-<wire x1="2.1154" y1="7" x2="6" y2="7" width="2.4" layer="1"/>
 <wire x1="6" y1="7" x2="8.8" y2="7" width="2.4" layer="1"/>
 <wire x1="8.8" y1="7" x2="10.9" y2="7" width="0.6096" layer="1"/>
 <wire x1="6" y1="6.45" x2="6" y2="7" width="0.6096" layer="1"/>
+<contactref element="J$1" pad="SIG"/>
+<wire x1="6" y1="7" x2="2.46" y2="7" width="2.4" layer="1"/>
+<wire x1="2.46" y1="7" x2="2.4" y2="6.99" width="2.4" layer="1"/>
 </signal>
 <signal name="N$2" class="1">
@@
 </signal>
 <signal name="N$6" class="1">
-<contactref element="RFOUT" pad="1"/>
 <contactref element="IC2" pad="7"/>
 <wire x1="28.9" y1="7.05" x2="30.95" y2="7.05" width="0.3" layer="1"/>
 <wire x1="30.95" y1="7.05" x2="31" y2="7" width="0.3" layer="1"/>
-<wire x1="31" y1="7" x2="37.8846" y2="7" width="2.4" layer="1"/>
+<contactref element="J$2" pad="SIG"/>
+<wire x1="31" y1="7" x2="37.59" y2="7" width="2.4" layer="1"/>
+<wire x1="37.59" y1="7" x2="37.6" y2="6.99" width="2.4" layer="1"/>
 </signal>
 <signal name="+5V">
